Commit message: Add Apriltag model in Gazebo

File: src/Env/husky/husky_description/urdf/husky.urdf.xacro (robot description, xacro)
@@ -255,5 +255,5 @@
   </joint>
   <gazebo reference="apriltag0_link">
-    <material>Apriltag</material>
+    <material>Apriltag0</material>
   </gazebo>
   <gazebo><plugin filename="libgazebo_ros_p3d.so" name="quadrotor_groundtruth_sim">

Commit message: Add plugin for rotor simulation to test_room.world

File: src/Env/husky/husky_description/urdf/husky.urdf.xacro (robot description, xacro)
@@ -255,5 +255,5 @@
   </joint>
   <gazebo reference="apriltag0_link">
-    <material>Apriltag0</material>
+    <material>Apriltag</material>
   </gazebo>
   <gazebo><plugin filename="libgazebo_ros_p3d.so" name="quadrotor_groundtruth_sim">

File: src/Env/multirotor_geometry_control/rotors_simulator/rotors_description/urdf/_d435.urdf.xacro (robot description, xacro)
@@ -61,5 +61,5 @@
       <inertial>
         <!-- The following are not reliable values, and should not be used for modeling -->
-        <mass value="0.564" />
+        <mass value="0.00001" />
         <origin xyz="0 0 0" />
         <inertia ixx="0.003881243" ixy="0.0" ixz="0.0" iyy="0.000498940" iyz="0.0" izz="0.003879257" />
